File: Hardware/Backplane Pro/Rev 1.0/Backplane Pro.kicad_pcb (KiCad board)
At the start: 2 copper layers, 100 x 100 mm, 49 parts, among them J1 PWR_SW, J10 6502 Bus, J2 USB_C_Receptacle_USB2.0, J3 RESET_SW, J4 CLOCK_ENBL_SW, J5 6502 Card Connector, J6 6502 Card Connector, J7 6502 Card Connector, J8 6502 Card Connector, J9 6502 Card Connector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

Commit message: Project restructuring
Connections:
- J2 pad S1: GND -> (no net)
