File: Hardware/CPU Card Pro/Rev 1.0/CPU Card Pro.kicad_pcb (KiCad board)
At the start: 2 copper layers, 100 x 57.6 mm, 20 parts, among them J1 6502 Card Edge, J2 BANK ADDR, J3 EXP, U1 65C816, U2 74HC00, U3 74HC245, U4 74HC573

Commit message: Change pull up resistor values
Parts:
- R1, R2, R3, R4, R5, R6: value 1k -> 10k
