File: Hardware/DB25 Helper/Rev 1.0/DB25 Helper.kicad_pcb (KiCad board)
At the start: 2 copper layers, 100 x 50 mm, 10 parts, among them J1 PORT A, J2 PORT B, J3 KEYBOARD

Commit message: Add BOMs to README
Connections:
- J3 pad SH: (no net) -> GND
