File: Hardware/Keyboard Helper/Rev 1.0/Keyboard Helper.kicad_pcb (KiCad board)
At the start: 2 copper layers, 335 x 125 mm, 101 parts, among them J1 JOYSTICK A, J2 JOYSTICK B, J3 JOYSTICK A, J4 JOYSTICK B, J5 PORT A, J6 PORT B, J7 KEYBOARD, SW1 `, SW10 9, SW11 0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

Commit message: Add BOMs to README
Connections:
- J1 pad SH: (no net) -> GND
- J2 pad SH: (no net) -> GND
- J7 pad SH: (no net) -> GND
