File: Hardware/Prototype Card/Rev 1.0/Prototype Card.kicad_sch (KiCad schematic)
At the start: 7 parts, among them J1 6502 Card Edge, J2 Conn_02x20_Odd_Even, J3 Conn_02x04_Odd_Even, U1 74HC138

Commit message: Project restructuring
Connections:
- net A0: now also J2.37 (Pin_37); no longer J2.38 (Pin_38)
- net A1: now also J2.35 (Pin_35); no longer J2.36 (Pin_36)
- net A10: now also J2.17 (Pin_17); no longer J2.18 (Pin_18)
- net A11: now also J2.15 (Pin_15); no longer J2.16 (Pin_16)
- net A12: now also J2.13 (Pin_13); no longer J2.14 (Pin_14)
- net A13: now also J2.11 (Pin_11); no longer J2.12 (Pin_12)
- net A14: now also J2.9 (Pin_9); no longer J2.10 (Pin_10)
- net A15: now also J2.7 (Pin_7); no longer J2.8 (Pin_8)
- net A2: now also J2.33 (Pin_33); no longer J2.34 (Pin_34)
- net A3: now also J2.31 (Pin_31); no longer J2.32 (Pin_32)
- net A4: now also J2.29 (Pin_29); no longer J2.30 (Pin_30)
- net A5: now also J2.27 (Pin_27); no longer J2.28 (Pin_28)
- net A6: now also J2.25 (Pin_25); no longer J2.26 (Pin_26)
- net A7: now also J2.23 (Pin_23); no longer J2.24 (Pin_24)
- net A8: now also J2.21 (Pin_21); no longer J2.22 (Pin_22)
- net A9: now also J2.19 (Pin_19); no longer J2.20 (Pin_20)
- net BE: now also J2.12 (Pin_12); no longer J2.11 (Pin_11)
- net D0: now also J2.38 (Pin_38); no longer J2.37 (Pin_37)
- net D1: now also J2.36 (Pin_36); no longer J2.35 (Pin_35)
- net D2: now also J2.34 (Pin_34); no longer J2.33 (Pin_33)
- net D3: now also J2.32 (Pin_32); no longer J2.31 (Pin_31)
- net D4: now also J2.30 (Pin_30); no longer J2.29 (Pin_29)
- net D5: now also J2.28 (Pin_28); no longer J2.27 (Pin_27)
- net D6: now also J2.26 (Pin_26); no longer J2.25 (Pin_25)
- net D7: now also J2.24 (Pin_24); no longer J2.23 (Pin_23)
- net EXP0: now also J2.5 (Pin_5); no longer J2.6 (Pin_6)
- net EXP1: now also J2.3 (Pin_3); no longer J2.4 (Pin_4)
- net EXP2: now also J2.22 (Pin_22); no longer J2.21 (Pin_21)
- net EXP3: now also J2.20 (Pin_20); no longer J2.19 (Pin_19)
- net GND: now also J2.2 (Pin_2), J2.39 (Pin_39); no longer J2.1 (Pin_1), J2.40 (Pin_40)
- net IRQB: now also J2.6 (Pin_6); no longer J2.5 (Pin_5)
- net NMIB: now also J2.8 (Pin_8); no longer J2.7 (Pin_7)
- net PHI2: now also J2.18 (Pin_18); no longer J2.17 (Pin_17)
- net RDY: now also J2.10 (Pin_10); no longer J2.9 (Pin_9)
- net RESB: now also J2.4 (Pin_4); no longer J2.3 (Pin_3)
- net RWB: now also J2.14 (Pin_14); no longer J2.13 (Pin_13)
- net SYNC: now also J2.16 (Pin_16); no longer J2.15 (Pin_15)
- net VCC: now also J2.1 (Pin_1), J2.40 (Pin_40); no longer J2.2 (Pin_2), J2.39 (Pin_39)

Commit message: Add BOMs
Parts:
- J2, J3: now in the parts list
Changed lines of the file:
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@@
 		(body_style 1)
 		(exclude_from_sim no)
-		(in_bom no)
+		(in_bom yes)
 		(on_board yes)
 		(in_pos_files yes)
@@
 		(body_style 1)
 		(exclude_from_sim no)
-		(in_bom no)
+		(in_bom yes)
 		(on_board yes)
 		(in_pos_files yes)

Commit message: Add BOMs to README
Parts:
- J2, J3: now left out of the parts list
Changed lines of the file:
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@@
 		(body_style 1)
 		(exclude_from_sim no)
-		(in_bom yes)
+		(in_bom no)
 		(on_board yes)
 		(in_pos_files yes)
@@
 		(body_style 1)
 		(exclude_from_sim no)
-		(in_bom yes)
+		(in_bom no)
 		(on_board yes)
 		(in_pos_files yes)
