File: Hardware/Serial Card Pro/Rev 1.0/Serial Card Pro.kicad_pcb (KiCad board)
At the start: 2 copper layers, 100 x 57.6 mm, 30 parts, among them J1 6502 Card Edge, J2 DB9 MALE (DTE), J3 Conn_02x08_Odd_Even, J4 DCD Select, U1 MAX232, U2 MAX232, U3 74HC138, U4 6551, Y1 1.8432 Mhz

Commit message: Project restructuring
Parts:
- J2: footprint 6502 Parts:DB9 Male -> Connector_Dsub:DSUB-9_Pins_Horizontal_P2.77x2.84mm_EdgePinOffset7.70mm_Housed_MountingHolesOffset9.12mm
