File: Hardware/Storage Card/Rev 1.0/Storage Card.kicad_pcb (KiCad board)
At the start: 2 copper layers, 100 x 57.6 mm, 18 parts, among them J1 6502 Card Edge, J2 Conn_02x08_Odd_Even, J3 Compact Flash, J4 ACT LED, U1 74HC00, U2 74HC138

Commit message: Schematic fix
Connections:
- net ~{RD} renamed RB
- net ~{WR} renamed WB
