File: Hardware/CPU Card/Rev 1.1/CPU Card.kicad_pcb (KiCad board)
At the start: 2 copper layers, 100 x 57.6 mm, 15 parts, among them J1 6502 Card Edge, J2 Conn_01x02, J3 EXP, U1 65C02

Commit message: Add CPU Card Rev 1.1
Parts:
- R1, R2, R3, R4, R5, R6: value 1k -> 10k
Other:
- board text added: "© 2024 A.C. Wright Design | acwrightdesign.com | Rev 1.1"
- board text removed: "© 2024 A.C. Wright Design | acwrightdesign.com | Rev 1.0"
