File: Hardware/CPU Card/Rev 1.1/CPU Card.kicad_sch (KiCad schematic)
At the start: 12 parts, among them J1 6502 Card Edge, J2 Conn_01x02, J3 EXP, U1 65C02

Commit message: Add CPU Card Rev 1.1
Parts:
- J2, J3, U1: now left out of the parts list
- R1, R2, R3, R4, R5, R6: value 1k -> 10k; LCSC C17513 -> C2930231
Changed lines of the file:
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@@
 		(title "6502 CPU Card")
 		(date "2024-07-03")
-		(rev "1.0")
+		(rev "1.1")
 		(company "A.C. Wright Design")
 	)
@@
 		(body_style 1)
 		(exclude_from_sim no)
-		(in_bom yes)
+		(in_bom no)
 		(on_board yes)
 		(in_pos_files yes)
@@
 			)
 		)
-		(property "Value" "1k"
+		(property "Value" "10k"
 			(at 208.28 50.3936 90)
 			(show_name no)
@@
 			)
 		)
-		(property "LCSC" "C17513"
+		(property "LCSC" "C2930231"
 			(at 208.28 53.34 0)
 			(hide yes)
@@
 			)
 		)
-		(property "Value" "1k"
+		(property "Value" "10k"
 			(at 208.28 58.0136 90)
 			(show_name no)
@@
 			)
 		)
-		(property "LCSC" "C17513"
+		(property "LCSC" "C2930231"
 			(at 208.28 60.96 0)
 			(hide yes)
@@
 			)
 		)
-		(property "Value" "1k"
+		(property "Value" "10k"
 			(at 208.28 65.6336 90)
 			(show_name no)
@@
 			)
 		)
-		(property "LCSC" "C17513"
+		(property "LCSC" "C2930231"
 			(at 208.28 68.58 0)
 			(hide yes)
@@
 			)
 		)
-		(property "Value" "1k"
+		(property "Value" "10k"
 			(at 208.28 73.2536 90)
 			(show_name no)
@@
 			)
 		)
-		(property "LCSC" "C17513"
+		(property "LCSC" "C2930231"
 			(at 208.28 76.2 0)
 			(hide yes)
@@
 			)
 		)
-		(property "Value" "1k"
+		(property "Value" "10k"
 			(at 208.28 80.8736 90)
 			(show_name no)
@@
 			)
 		)
-		(property "LCSC" "C17513"
+		(property "LCSC" "C2930231"
 			(at 208.28 83.82 0)
 			(hide yes)
@@
 		(body_style 1)
 		(exclude_from_sim no)
-		(in_bom yes)
+		(in_bom no)
 		(on_board yes)
 		(in_pos_files yes)
@@
 			)
 		)
-		(property "Value" "1k"
+		(property "Value" "10k"
 			(at 208.28 88.4936 90)
 			(show_name no)
@@
 			)
 		)
-		(property "LCSC" "C17513"
+		(property "LCSC" "C2930231"
 			(at 208.28 91.44 0)
 			(hide yes)
@@
 		(body_style 1)
 		(exclude_from_sim no)
-		(in_bom yes)
+		(in_bom no)
 		(on_board yes)
 		(in_pos_files yes)
